File: core/core.kicad_pcb (KiCad board)
At the start: 2 copper layers, 99.7 x 98.4 mm, 55 parts, among them J1 HC-05, J10 AUX1, J11 AUX2, J12 AUX3, J13 AUX4, J14 DIST_IZQ, J15 DIST_FRONT, J16 DIST_DCHA, J2 TB6612FNG_A, J3 MOT_IZQ, J4 MOT_DER, J5 TB6612FNG_B, J6 LIPO_2S, J7 Sensores_linea, J8 LIPO_1S_A, J9 LIPO_1S_B, SW1 B1, SW2 B2, SW3 SW_DPDT_x2, U1 Arduino_Nano_v3.x, U2 DC-DC_BuckModule, U3 PCF8574

Commit message: Gerbers exportados y mandado a fabrica
Parts:
- added G***: LOGO, logos:logaso, B.Cu at (202.1, 128.8)
- added G***: LOGO, logos:logaso, F.Cu at (202.1, 129.2)
- added G***: LOGO, logos:tortu, B.Cu at (201.3, 74.4)
- renumbered J6 to 2S_Bat, J8 to A, J9 to B, SW1 to B1, SW2 to B2, J16 to DIS_DER, J15 to DIS_FRONT, J14 to DIS_IZQ, J4 to M_Dr, J3 to M_Iz, J7 to Sensores
Routing:
- net +5V: track 378.6 -> 380.1 mm
Other:
- board text added: "+"
- board text added: "2 x 1S Bat"
- board text added: "5V"
- board text added: "A1"
- board text added: "D10"
- board text added: "D11"
- board text added: "D13"
- board text added: "D7"
- board text added: "D8"
- board text added: "D9"
- board text added: "GND"
- board text added: "L1"
- board text added: "L2"
- board text added: "L3"
- board text added: "L_S"
- board text added: "OFF"
- board text added: "ON"
