File: core/core.sch (KiCad schematic (older format))
At the start: 39 parts, among them J1 HC-05, J10 AUX1, J11 AUX2, J12 AUX3, J13 AUX4, J14 DIST_IZQ, J15 DIST_FRONT, J16 DIST_DCHA, J2 TB6612FNG_A, J3 MOT_IZQ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

Commit message: Pdfs exportados
Parts:
- C1, C2: symbol device:C_Small -> core-rescue:C_Small-device
- D1, D3: symbol LED:NeoPixel_THT -> core-rescue:NeoPixel_THT-LED
- D2, D6: symbol device:D_Small -> core-rescue:D_Small-device
- D4, D5: symbol device:LED_Small -> core-rescue:LED_Small-device
- J1, J7: symbol Connector_Generic:Conn_01x06 -> core-rescue:Conn_01x06-Connector_Generic
- J10, J11, J12, J13, J14, J15, J16, J6: symbol Connector_Generic:Conn_01x03 -> core-rescue:Conn_01x03-Connector_Generic
- J2, J5: symbol Connector_Generic:Conn_01x08 -> core-rescue:Conn_01x08-Connector_Generic
- J3, J4, J8, J9: symbol Connector_Generic:Conn_01x02 -> core-rescue:Conn_01x02-Connector_Generic
- JP1: symbol device:Jumper_NO_Small -> core-rescue:Jumper_NO_Small-device
- R1, R2, R3, R4, R5, R6, R7, R8: symbol device:R_Small -> core-rescue:R_Small-device
- U1: symbol MCU_Module:Arduino_Nano_v3.x -> core-rescue:Arduino_Nano_v3.x-MCU_Module
- U2: symbol DC-DC_MP2307:DC-DC_BuckModule -> core-rescue:DC-DC_BuckModule-DC-DC_MP2307
- U3: symbol Interface_Expansion:PCF8574 -> core-rescue:PCF8574-Interface_Expansion
Changed lines of the file:
@@
 $EndDescr
 $Comp
-L MCU_Module:Arduino_Nano_v3.x U1
+L core-rescue:Arduino_Nano_v3.x-MCU_Module U1
 U 1 1 5BF4DDE4
 P 3950 2400
@@
 $EndComp
 $Comp
-L device:R_Small R3
+L core-rescue:R_Small-device R3
 U 1 1 5BF516C0
 P 8550 1550
@@
 $EndComp
 $Comp
-L device:R_Small R4
+L core-rescue:R_Small-device R4
 U 1 1 5BF5188E
 P 8900 1550
@@
 	8550 1700 8550 1650
 $Comp
-L device:R_Small R1
+L core-rescue:R_Small-device R1
 U 1 1 5BF5C75C
 P 7400 1650
@@
 $EndComp
 $Comp
-L device:R_Small R2
+L core-rescue:R_Small-device R2
 U 1 1 5BF5C8B8
 P 7750 1650
@@
 $EndComp
 $Comp
-L device:LED_Small D4
+L core-rescue:LED_Small-device D4
 U 1 1 5BF5CB11
 P 7400 1950
@@
 $EndComp
 $Comp
-L device:LED_Small D5
+L core-rescue:LED_Small-device D5
 U 1 1 5BF5CC19
 P 7750 1950
@@
 B2
 $Comp
-L Connector_Generic:Conn_01x08 J2
+L core-rescue:Conn_01x08-Connector_Generic J2
 U 1 1 5BF6E2AD
 P 3950 5950
@@
 $EndComp
 $Comp
-L Connector_Generic:Conn_01x08 J5
+L core-rescue:Conn_01x08-Connector_Generic J5
 U 1 1 5BF703F5
 P 4400 5950
@@
 M_DER_+
 $Comp
-L Connector_Generic:Conn_01x02 J3
+L core-rescue:Conn_01x02-Connector_Generic J3
 U 1 1 5BFAC6C5
 P 4350 6650
@@
 $EndComp
 $Comp
-L Connector_Generic:Conn_01x02 J4
+L core-rescue:Conn_01x02-Connector_Generic J4
 U 1 1 5BFAC979
 P 4350 6950
@@
 MOTORES
 $Comp
-L LED:NeoPixel_THT D1
+L core-rescue:NeoPixel_THT-LED D1
 U 1 1 5BFCA810
 P 1250 6650
@@
 $EndComp
 $Comp
-L Connector_Generic:Conn_01x06 J1
+L core-rescue:Conn_01x06-Connector_Generic J1
 U 1 1 5BFCB80B
 P 2100 4350
@@
 $EndComp
 $Comp
-L device:R_Small R5
+L core-rescue:R_Small-device R5
 U 1 1 5BFCEB26
 P 5850 6100
@@
 $EndComp
 $Comp
-L device:R_Small R6
+L core-rescue:R_Small-device R6
 U 1 1 5BFCECB3
 P 5850 6450
@@
 	5850 6000 5850 5850
 $Comp
-L device:D_Small D6
+L core-rescue:D_Small-device D6
 U 1 1 5BFDD5C4
 P 6300 6100
@@
 	6300 5850 6300 6000
 $Comp
-L LED:NeoPixel_THT D3
+L core-rescue:NeoPixel_THT-LED D3
 U 1 1 5BFE9C91
 P 2150 6650
@@
 BT_RX
 $Comp
-L device:D_Small D2
+L core-rescue:D_Small-device D2
 U 1 1 5BF7351E
 P 1450 4450
@@
 NEOPIXELS
 $Comp
-L device:C_Small C1
+L core-rescue:C_Small-device C1
 U 1 1 5BF95CD1
 P 1500 6300
@@
 $EndComp
 $Comp
-L device:C_Small C2
+L core-rescue:C_Small-device C2
 U 1 1 5BF95F64
 P 2400 6300
@@
 PULSADORES
 $Comp
-L Connector_Generic:Conn_01x02 J8
+L core-rescue:Conn_01x02-Connector_Generic J8
 U 1 1 5BFCB48F
 P 6550 1450
@@
 $EndComp
 $Comp
-L Connector_Generic:Conn_01x03 J6
+L core-rescue:Conn_01x03-Connector_Generic J6
 U 1 1 5BFCB6C2
 P 5550 1650
@@
 $EndComp
 $Comp
-L Connector_Generic:Conn_01x02 J9
+L core-rescue:Conn_01x02-Connector_Generic J9
 U 1 1 5BF59BEA
 P 6550 1750
@@
 STBY_MOT
 $Comp
-L DC-DC_MP2307:DC-DC_BuckModule U2
+L core-rescue:DC-DC_BuckModule-DC-DC_MP2307 U2
 U 1 1 5BF9CA8B
 P 10200 3600
@@
 $EndComp
 $Comp
-L Connector_Generic:Conn_01x06 J7
+L core-rescue:Conn_01x06-Connector_Generic J7
 U 1 1 5BF569B8
 P 7500 5450
@@
 BT_RX
 $Comp
-L Interface_Expansion:PCF8574 U3
+L core-rescue:PCF8574-Interface_Expansion U3
 U 1 1 5BFDA0BA
 P 6700 4000
@@
 	7300 4300 7200 4300
 $Comp
-L device:R_Small R8
+L core-rescue:R_Small-device R8
 U 1 1 5C02A571
 P 6100 3400
@@
 $EndComp
 $Comp
-L device:R_Small R7
+L core-rescue:R_Small-device R7
 U 1 1 5C02A7C3
 P 5950 3400
@@
 NEO
 $Comp
-L Connector_Generic:Conn_01x03 J14
+L core-rescue:Conn_01x03-Connector_Generic J14
 U 1 1 5C06B480
 P 8400 5850
@@
 $EndComp
 $Comp
-L Connector_Generic:Conn_01x03 J15
+L core-rescue:Conn_01x03-Connector_Generic J15
 U 1 1 5C072223
 P 9350 5850
@@
 $EndComp
 $Comp
-L Connector_Generic:Conn_01x03 J16
+L core-rescue:Conn_01x03-Connector_Generic J16
 U 1 1 5C07252F
 P 10300 5850
@@
 SENSORES
 $Comp
-L Connector_Generic:Conn_01x03 J10
+L core-rescue:Conn_01x03-Connector_Generic J10
 U 1 1 5C18209A
 P 1150 2450
@@
 $EndComp
 $Comp
-L Connector_Generic:Conn_01x03 J11
+L core-rescue:Conn_01x03-Connector_Generic J11
 U 1 1 5C182515
 P 1150 3000
@@
 $EndComp
 $Comp
-L Connector_Generic:Conn_01x03 J12
+L core-rescue:Conn_01x03-Connector_Generic J12
 U 1 1 5C1827FE
 P 1950 2450
@@
 $EndComp
 $Comp
-L Connector_Generic:Conn_01x03 J13
+L core-rescue:Conn_01x03-Connector_Generic J13
 U 1 1 5C182954
 P 1950 3000
@@
 	9250 4200 9800 4200
 $Comp
-L device:Jumper_NO_Small JP1
+L core-rescue:Jumper_NO_Small-device JP1
 U 1 1 5BF9B713
 P 9900 4200
