File: sensores/sensores.sch (KiCad schematic (older format))
At the start: 17 parts, among them J1 Conn_01x06_Female, U1 CNY70, U2 CNY70, U3 CNY70, U4 CNY70, U5 CNY70, U6 CNY70, U7 4053

Commit message: Pdfs exportados
Parts:
- R1, R2, R3, R4, R5, R6, R7, R8, R9: symbol Device:R_Small -> sensores-rescue:R_Small-Device
- U1, U2, U3, U4, U5, U6: symbol Sensor_Proximity:CNY70 -> sensores-rescue:CNY70-Sensor_Proximity
- U7: symbol 4xxx:4053 -> sensores-rescue:4053-4xxx
Changed lines of the file:
@@
 $EndDescr
 $Comp
-L Sensor_Proximity:CNY70 U1
+L sensores-rescue:CNY70-Sensor_Proximity U1
 U 1 1 5BEFF17C
 P 2500 2750
@@
 $EndComp
 $Comp
-L Sensor_Proximity:CNY70 U2
+L sensores-rescue:CNY70-Sensor_Proximity U2
 U 1 1 5BEFF1E8
 P 2500 3950
@@
 $EndComp
 $Comp
-L Sensor_Proximity:CNY70 U3
+L sensores-rescue:CNY70-Sensor_Proximity U3
 U 1 1 5BEFF251
 P 4000 2750
@@
 $EndComp
 $Comp
-L Sensor_Proximity:CNY70 U4
+L sensores-rescue:CNY70-Sensor_Proximity U4
 U 1 1 5BEFF2A8
 P 4000 3950
@@
 $EndComp
 $Comp
-L Sensor_Proximity:CNY70 U5
+L sensores-rescue:CNY70-Sensor_Proximity U5
 U 1 1 5BEFF46A
 P 5450 2750
@@
 $EndComp
 $Comp
-L Sensor_Proximity:CNY70 U6
+L sensores-rescue:CNY70-Sensor_Proximity U6
 U 1 1 5BEFF4E5
 P 5450 3950
@@
 $EndComp
 $Comp
-L Device:R_Small R5
+L sensores-rescue:R_Small-Device R5
 U 1 1 5BEFFC2F
 P 4350 3650
@@
 $EndComp
 $Comp
-L Device:R_Small R9
+L sensores-rescue:R_Small-Device R9
 U 1 1 5BEFFEB6
 P 5800 3650
@@
 $EndComp
 $Comp
-L Device:R_Small R3
+L sensores-rescue:R_Small-Device R3
 U 1 1 5BF00134
 P 2900 2450
@@
 $EndComp
 $Comp
-L Device:R_Small R6
+L sensores-rescue:R_Small-Device R6
 U 1 1 5BF00244
 P 4400 2450
@@
 $EndComp
 $Comp
-L Device:R_Small R8
+L sensores-rescue:R_Small-Device R8
 U 1 1 5BF00499
 P 5800 2450
@@
 $EndComp
 $Comp
-L Device:R_Small R2
+L sensores-rescue:R_Small-Device R2
 U 1 1 5BF00725
 P 2850 3650
@@
 	2150 2850 2150 3250
 $Comp
-L Device:R_Small R1
+L sensores-rescue:R_Small-Device R1
 U 1 1 5BF17DCF
 P 2150 3350
@@
 	2150 3450 2150 3850
 $Comp
-L Device:R_Small R4
+L sensores-rescue:R_Small-Device R4
 U 1 1 5BF1945C
 P 3600 3350
@@
 sensor6
 $Comp
-L Device:R_Small R7
+L sensores-rescue:R_Small-Device R7
 U 1 1 5BF1F998
 P 5050 3350
@@
 	5050 2850 5050 3250
 $Comp
-L 4xxx:4053 U7
+L sensores-rescue:4053-4xxx U7
 U 1 1 5BF23F0F
 P 8550 4650
